File: NanoPi-R4S-spi-flash-module.sch (KiCad schematic (older format))
At the start: 22 parts, among them J1 NanoPi R4S, J2 TagConnect_TC2030_SWD, U1 W25Q32JVSS, U2 MX25R3235FZNxx0, U3 W25Q32JVSS, U4 MX25R3235FZNxx0, U5 STM32G031GxU

Commit message: Replace D1 by regular silicon diode
Schottky diodes tend to have high leakage current. Considering the MCU is
supposed to be kept running on C4 and C5 as long as possible after power
has been removed reducing leakage current back into the 3.3V supply rail
is key.
Replace D1 by an ordinary 1N4148 to minimize leakage current back into the
3.3V supply rail.
Parts:
- D1: value B5819W -> 1N4148W; symbol Device:D_Schottky -> Device:D; LCSC C8598 -> C81598
Changed lines of the file:
@@
 	8550 2300 8550 3050
 $Comp
-L Device:D_Schottky D1
+L Device:D D1
 U 1 1 61C64DB7
 P 6000 1750
 F 0 "D1" H 6000 1533 50  0000 C CNN
-F 1 "B5819W" H 6000 1624 50  0000 C CNN
+F 1 "1N4148W" H 6000 1624 50  0000 C CNN
 F 2 "Diode_SMD:D_SOD-123" H 6000 1750 50  0001 C CNN
 F 3 "~" H 6000 1750 50  0001 C CNN
-F 4 "C8598" H 6000 1750 50  0001 C CNN "LCSC"
+F 4 "C81598" H 6000 1750 50  0001 C CNN "LCSC"
 	1    6000 1750
 	-1   0    0    1
@@
 NoConn ~ 6600 3100
 $Comp
-L power:PWR_FLAG #FLG?
+L power:PWR_FLAG #FLG0101
 U 1 1 61D3185B
 P 7250 1750
-F 0 "#FLG?" H 7250 1825 50  0001 C CNN
+F 0 "#FLG0101" H 7250 1825 50  0001 C CNN
 F 1 "PWR_FLAG" H 7250 1923 50  0000 C CNN
 F 2 "" H 7250 1750 50  0001 C CNN
@@
 Connection ~ 7250 1750
 $Comp
-L power:PWR_FLAG #FLG?
+L power:PWR_FLAG #FLG0102
 U 1 1 61D3209B
 P 2100 1350
-F 0 "#FLG?" H 2100 1425 50  0001 C CNN
+F 0 "#FLG0102" H 2100 1425 50  0001 C CNN
 F 1 "PWR_FLAG" H 2100 1523 50  0000 C CNN
 F 2 "" H 2100 1350 50  0001 C CNN
@@
 Connection ~ 1800 1600
 $Comp
-L power:PWR_FLAG #FLG?
+L power:PWR_FLAG #FLG0103
 U 1 1 61D34E55
 P 900 1350
-F 0 "#FLG?" H 900 1425 50  0001 C CNN
+F 0 "#FLG0103" H 900 1425 50  0001 C CNN
 F 1 "PWR_FLAG" H 900 1523 50  0000 C CNN
 F 2 "" H 900 1350 50  0001 C CNN
@@
 Connection ~ 1200 1500
 $Comp
-L power:GND #PWR?
+L power:GND #PWR0129
 U 1 1 61D38819
 P 10650 1250
-F 0 "#PWR?" H 10650 1000 50  0001 C CNN
+F 0 "#PWR0129" H 10650 1000 50  0001 C CNN
 F 1 "GND" H 10655 1077 50  0000 C CNN
 F 2 "" H 10650 1250 50  0001 C CNN
@@
 $EndComp
 $Comp
-L power:PWR_FLAG #FLG?
+L power:PWR_FLAG #FLG0104
 U 1 1 61D38FF5
 P 10650 1200
-F 0 "#FLG?" H 10650 1275 50  0001 C CNN
+F 0 "#FLG0104" H 10650 1275 50  0001 C CNN
 F 1 "PWR_FLAG" H 10650 1373 50  0000 C CNN
 F 2 "" H 10650 1200 50  0001 C CNN
