File: NanoPi-R4S-spi-flash-module.kicad_pcb (KiCad board)
At the start: 4 copper layers, 30 x 13.2 mm, 22 parts, among them J1 NanoPi R4S, J2 TagConnect_TC2030_SWD, U1 W25Q32JVSS, U2 MX25R3235FZNxx0, U3 W25Q32JVSS, U4 MX25R3235FZNxx0, U5 STM32G031GxU

Commit message: Fix incorrect MCU partnumber
Parts:
- turned C7 to 0 degrees
Connections:
- net /FLASH_~RST renamed /FLASH_~{RST}
- net /FLASH_~WP renamed /FLASH_~{WP}
- net /SPI1_~CS renamed /SPI1_~{CS}
- net /~RST renamed /~{RST}
Routing:
- net /FLASH_~{RST}: track 25.7 -> 25.1 mm, vias 3 -> 2
- net GND: track 10.7 -> 11.4 mm, vias 10 -> 11
Other:
- net class Default removed
- board text added: "NanoPi R4S NOR flash Designed by Tobias Schramm Rev 1.1 2021"
- board text removed: "NanoPi R4S NOR flash Designed by Tobias Schramm Rev 1.0 2021"
